File: hardware/handbell/handbell.kicad_sch (KiCad schematic)
At the start: 82 parts, among them IC1 RP2040_QFN56, IC2 74AHCT1G125DCK, IC4 LSM6DSOXTR, Q1 AO3401, Q2 C20917, Q3 DMG3415UFY, SW1 RKB2, SW2 RKB2, U1 8MB QSPI, U2 RT9080-3.3, U3 MCP73831T-2ACI/OT, U4 MAX98357A, X1 JSTPH, X6 USB Type C, Y1 12MHz/12pF

Commit message: Add reduced handbell electronics and printable fit-study kit
Implement the licensed TPS61023 boost, mute/button and connector reduction; preserve explicit electrical and native placement evidence. Add the 43 mm unrouted candidate, editable FreeCAD assembly, populated-PCBA/speaker/battery fit dummies, and PLA/routing handoffs. Retain unresolved power, USB, mechanical and fabrication gates.

Co-authored-by: Copilot <223556219+Copilot@users.noreply.github.com>
Parts:
- removed CONN1: STEMMA_I2C_QTRA, Adafruit Feather RP2040 Prop-Maker-import-fps:JST_SH4_RA, symbol Handbell:STEMMA_I2C_QTRA
- removed IC2: 74AHCT1G125DCK, Adafruit Feather RP2040 Prop-Maker-import-fps:SC70-5, symbol Handbell:741G125DCKAHCT
- removed JP1: HEADER-1X16ROUND, Adafruit Feather RP2040 Prop-Maker-import-fps:1X16_ROUND, symbol Handbell:HEADER-1X16ROUND
- removed JP3: HEADER-1X12, Adafruit Feather RP2040 Prop-Maker-import-fps:1X12_ROUND, symbol Handbell:HEADER-1X12
- removed LED1: WS2812B_SK6805_1515, Adafruit Feather RP2040 Prop-Maker-import-fps:SK6805_1515, symbol Handbell:WS2812B_SK6805_1515
- removed OUTPUTS0: TERMINALS, Adafruit Feather RP2040 Prop-Maker-import-fps:1X06_OVAL, symbol Handbell:HEADER-1X6
- removed R19: 100, Adafruit Feather RP2040 Prop-Maker-import-fps:_0402NO, symbol Handbell:RESISTOR_0402NO
- removed SERVO0: 1x3M, Adafruit Feather RP2040 Prop-Maker-import-fps:1X03_ROUND_76, symbol Handbell:HEADER-1X376MIL
- removed SW1, SW2: RKB2, Adafruit Feather RP2040 Prop-Maker-import-fps:BTN_RKB2_4.6X2.8, symbol Handbell:SWITCH_TACT_SMT_RKB2
- removed U$31, U$32: MOUNTINGHOLE2.5, Adafruit Feather RP2040 Prop-Maker-import-fps:MOUNTINGHOLE_2.5_PLATED, symbol Handbell:MOUNTINGHOLE2.5
- removed U$34, U$35: FIDUCIAL_1MM, Adafruit Feather RP2040 Prop-Maker-import-fps:FIDUCIAL_1MM, symbol Handbell:FIDUCIAL_1MM
- added C25: 10nF, Adafruit Feather RP2040 Prop-Maker-import-fps:_0402NO, symbol Handbell:CAP_CERAMIC_0402NO
- added C26, C27, C28: 22uF, Adafruit Feather RP2040 Prop-Maker-import-fps:0805-NO, symbol Handbell:CAP_CERAMIC0805-NOOUTLINE
- added C29: 220pF (DNP), Adafruit Feather RP2040 Prop-Maker-import-fps:_0402NO, symbol Handbell:CAP_CERAMIC_0402NO
- added J1: 504050-0291, Connector_Molex:Molex_Pico-Lock_504050-0291_1x02-1MP_P1.50mm_Horizontal, symbol Handbell:CONNECTOR_2
- added J2: SM02B-SRSS-TB, Connector_JST:JST_SH_SM02B-SRSS-TB_1x02-1MP_P1.00mm_Horizontal, symbol Handbell:CONNECTOR_2
- added L1: 1uH (MPN pending), Adafruit TPS61023-import-fps:INDUCTOR_5X5MM_TDK_VLC5045, symbol Handbell:INDUCTORTDK_VLC5045
- added Q4: AO3400A, Package_TO_SOT_SMD:SOT-23, symbol Handbell:MOSFET-NWIDE
- added R20: 4.7K, Adafruit Feather RP2040 Prop-Maker-import-fps:_0402NO, symbol Handbell:RESISTOR_0402NO
- added R21: 10K, Adafruit Feather RP2040 Prop-Maker-import-fps:_0402NO, symbol Handbell:RESISTOR_0402NO
- added R22: 1K, Adafruit Feather RP2040 Prop-Maker-import-fps:_0402NO, symbol Handbell:RESISTOR_0402NO
- added R23: 732K, Adafruit Feather RP2040 Prop-Maker-import-fps:_0402NO, symbol Handbell:RESISTOR_0402NO
- added R24: 100K, Adafruit Feather RP2040 Prop-Maker-import-fps:_0402NO, symbol Handbell:RESISTOR_0402NO
- added TP10: VAMP, Adafruit Feather RP2040 Prop-Maker-import-fps:TESTPOINT_ROUND_1.5MM_NO, symbol Handbell:TESTPOINTROUND1.5MMNO
- added TP11: VBAT, Adafruit Feather RP2040 Prop-Maker-import-fps:TESTPOINT_ROUND_1.5MM_NO, symbol Handbell:TESTPOINTROUND1.5MMNO
- added TP12: I2S_DIN, Adafruit Feather RP2040 Prop-Maker-import-fps:TESTPOINT_ROUND_1.5MM_NO, symbol Handbell:TESTPOINTROUND1.5MMNO
- added TP13: I2S_BCLK, Adafruit Feather RP2040 Prop-Maker-import-fps:TESTPOINT_ROUND_1.5MM_NO, symbol Handbell:TESTPOINTROUND1.5MMNO
- added TP14: I2S_LRCLK, Adafruit Feather RP2040 Prop-Maker-import-fps:TESTPOINT_ROUND_1.5MM_NO, symbol Handbell:TESTPOINTROUND1.5MMNO
- added TP15: AMP_MUTE, Adafruit Feather RP2040 Prop-Maker-import-fps:TESTPOINT_ROUND_1.5MM_NO, symbol Handbell:TESTPOINTROUND1.5MMNO
- added TP16: POWER, Adafruit Feather RP2040 Prop-Maker-import-fps:TESTPOINT_ROUND_1.5MM_NO, symbol Handbell:TESTPOINTROUND1.5MMNO
- added TP7: ~{RESET}, Adafruit Feather RP2040 Prop-Maker-import-fps:TESTPOINT_ROUND_1.5MM_NO, symbol Handbell:TESTPOINTROUND1.5MMNO
- added TP8: GND, Adafruit Feather RP2040 Prop-Maker-import-fps:TESTPOINT_ROUND_1.5MM_NO, symbol Handbell:TESTPOINTROUND1.5MMNO
- added TP9: +3V3, Adafruit Feather RP2040 Prop-Maker-import-fps:TESTPOINT_ROUND_1.5MM_NO, symbol Handbell:TESTPOINTROUND1.5MMNO
- added U5: TPS61023DRLR, Adafruit TPS61023-import-fps:SOT563, symbol Handbell:TPS61023
- CHG_EN0: footprint Adafruit Feather RP2040 Prop-Maker-import-fps:SOLDERJUMPER_CLOSEDWIRE -> Jumper:SolderJumper-2_P1.3mm_Bridged_Pad1.0x1.5mm; now left out of the parts list
- D+1, D-1, TP3, TP4, TP5, TP6: now left out of the parts list
- GAIN0: footprint Adafruit Feather RP2040 Prop-Maker-import-fps:SOLDERJUMPER_2WAY_OPEN_NOPASTE -> Jumper:SolderJumper-3_P1.3mm_Open_Pad1.0x1.5mm; now left out of the parts list
- Q3: footprint Adafruit Feather RP2040 Prop-Maker-import-fps:DFN2015-3 -> Handbell:DFN2015-3_DrainPad
- R18: value 1M -> 10K
Connections:
- net +3V3: now also R20.1, R21.1, TP9.P$1
- net BUTTON: now also C25.1, R21.2, R22.1
- net GND: now also C25.2, C26.2, C27.2, C28.2, J2.2, Q4.2 (S), R24.2, TP8.P$1, U5.4 (GND)
- net I2S_BCLK: now also TP13.P$1
- net I2S_DIN: now also TP12.P$1
- net I2S_LRCLK: now also TP14.P$1
- net I2S_MOD: now also Q4.3 (D)
- net POWER: now also TP16.P$1, U5.2 (EN)
- net V+: now also C26.1, L1.P$1 (1), U5.3 (VIN); no longer C16.1, C19.1, GAIN0.3, R18.2, U4.7 (VDD), U4.8 (VDD)
- net VBAT: now also TP11.P$1
- net VO+: now also J1.1
- net VO-: now also J1.2
- net ~{RESET}: now also TP7.P$1
- net A0: no longer names the net of IC1.38 (GPIO26/AD0)
- net A1: no longer names the net of IC1.39 (GPIO27/AD1)
- net A2: no longer names the net of IC1.40 (GPIO28/AD2)
- net A3: no longer names the net of IC1.41 (GPIO29/AD3)
- net D10: no longer names the net of IC1.13 (GPIO10)
- net D11: no longer names the net of IC1.14 (GPIO11)
- net D12: no longer names the net of IC1.15 (GPIO12)
- net D24: no longer names the net of IC1.36 (GPIO24)
- net D25: no longer names the net of IC1.37 (GPIO25)
- net D4: no longer names the net of IC1.6 (GPIO4)
- net D5: no longer names the net of IC1.7 (GPIO5)
- net D6: no longer names the net of IC1.8 (GPIO6)
- net D9: no longer names the net of IC1.12 (GPIO9)
- net MISO: no longer names the net of IC1.11 (GPIO8)
- net MOSI: no longer names the net of IC1.18 (GPIO15)
- net PIXELS: no longer names the net of IC1.32 (GPIO21)
- net RX: no longer names the net of IC1.3 (GPIO1)
- net SCK: no longer names the net of IC1.17 (GPIO14)
- net SERVO renamed AMP_MUTE
- net AMP_MUTE: now also Q4.1 (G), R20.2, TP15.P$1
- net TX: no longer names the net of IC1.2 (GPIO0)
- new net BOOST_FB: C29.2, R23.2, R24.1, U5.1 (FB)
- new net BOOST_SW: L1.P$2 (2), U5.5 (SW)
- new net BUTTON_EXT: J2.1, R22.2
- new net VAMP: C16.1, C19.1, C27.1, C28.1, C29.1, GAIN0.3, R18.2, R23.1, TP10.P$1, U4.7 (VDD), U4.8 (VDD), U5.6 (VOUT)
- no-connect marks 6 -> 24
Other:
- note added: "0.2 ELECTRICAL / PLACEMENT DRAFT - NOT FOR FABRICATION Cell, charge/temperature/cutoff policy and exact power MPNs unresolved. BTL speaker outputs: neither lead is ground. No hardware qualification."
- note added: "5V-CLASS AUDIO BOOST (Adafruit 4654-derived) EN follows GPIO23 POWER; existing R17 supplies default pulldown. R1 default-on pull-up omitted. Input remains behind Q1/Q2. Power MPNs / effective capacitance not frozen. C29: optional feed-forward; resolve for >40uF effective Cout."
- note added: "GPIO19 BUTTON HARNESS J2 -> 1K -> GPIO; 10K pull-up, 10nF filter. Firmware debounce + final cable/ESD review required."
- note added: "MONO LEFT + INDEPENDENT SHUTDOWN R18=10K to VAMP; Q4 pulls SD_MODE low. GPIO20 HIGH=mute, LOW=play; 9dB gain."
- note added: "POWER DECLARATIONS (not fitted parts) USB / return / mux / cell / switched input"
- note added: "Q4 / GPIO20: HIGH = SHUTDOWN 4.7K pull-up dominates RP2040 reset pulldown. Drive mute HIGH before enabling POWER. Supply collapse/pop behavior remains a bench gate."
- note added: "SERVICE PADS: no fitted headers; route to accessible edge/fixture. BOOT=TP3; RESET=TP7; SWCLK=TP4; SWDIO=TP5."
- note added: "SPEAKER: isolated BTL pair, 4 ohm target 3W high-end != qualified continuous speaker power. Molex Pico-Lock, not battery JST-PH or button JST-SH."
- note added: "STATUS LED (GPIO13)"
- note removed: "BREAKOUTS"
- note removed: "INTEGRATION DRAFT - NOT FOR FABRICATION Cell, charging temperature/current, speaker and quiet-idle behavior unresolved. BTL speaker outputs: neither lead is ground. Peripheral reduction pending."
- note removed: "NEOPIXEL"
- note removed: "Power-source declarations (not physical components) USB / return / discrete mux / external cell / switched rail"
- note removed: "R1 Channel Selection: LEFT = VDD (0 Ohm) RIGHT = 370K (94*VDD-100) LEFT/2 + RIGHT/2 = 1.011M (222.2*VDD-100)"
- note removed: "RED LED"
- note removed: "RESET"
- note removed: "SWD pads: add adjacent GND and 3V3 probe access at layout."
- title: Digital Handbell - LSM6DSOX integration draft -> Digital Handbell - compact boosted electrical draft
