File: hardware/handbell/iterations/printed-bell-clock-draft/handbell.kicad_sch (KiCad schematic)
At the start: 102 parts, among them IC1 RP2040_QFN56, IC4 LSM6DSOXTR, J1 504050-0291, J2 SM02B-SRSS-TB, Q1 AO3401, Q2 C20917, Q3 DMG3415UFY, Q4 AO3400A, Q5 CSD83325L, U1 W25Q16JVUXIQ TR / 2MB, U2 RT9080-3.3, U3 MCP73831T-2ACI/OT, U4 MAX98357A, U5 TPS61023DRLR, U6 BQ29700DSER, X6 USB Type C, Y1 12MHz/CL10pF

Commit message: Apply selected Q3 identity while retaining corrected native geometry
Preserve circuitry, copper and placements; publish scoped native identity and schematic evidence.

Co-authored-by: Copilot <223556219+Copilot@users.noreply.github.com>
Parts:
- Q3: value DMG3415UFY -> DMP2045UFY4; MPN (none) -> DMP2045UFY4-7; Manufacturer (none) -> Diodes Incorporated
Changed lines of the file:
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@@
 			)
 		)
-		(property "Value" "DMG3415UFY"
+		(property "Value" "DMP2045UFY4"
 			(at 51.054 41.275 0)
 			(show_name no)
@@
 			)
 		)
-		(property "Datasheet" ""
+		(property "Datasheet" "https://www.diodes.com/datasheet/download/DMP2045UFY4.pdf"
 			(at 48.26 43.18 0)
 			(hide yes)
@@
 			)
 		)
-		(property "Description" ""
+		(property "Description" "P-channel MOSFET; X2-DFN2015-3; G=1, S=2, D=3. Selected replacement, not electrically identical."
 			(at 48.26 43.18 0)
 			(hide yes)
@@
 			)
 		)
+(property "MPN" "DMP2045UFY4-7" (at 48.26 43.18 0)  (hide yes) (effects (font (size 1 1))))
+(property "Manufacturer" "Diodes Incorporated" (at 48.26 43.18 0)  (hide yes) (effects (font (size 1 1))))
 	)
 	(symbol

Commit message: Apply approved ordinary resistor identities without changing circuit values
Fill23 blank MPNs and confirm4; preserve circuit-reference links and all geometry/copper.

Co-authored-by: Copilot <223556219+Copilot@users.noreply.github.com>
Parts:
- R1, R14, R15, R18, R2, R21, R3, R4, R5, R7: MPN (none) -> RC0402FR-0710KL; Manufacturer (none) -> Yageo
- R10, R9: MPN (none) -> RC0402FR-0722RL; Manufacturer (none) -> Yageo
- R11, R22, R6: MPN (none) -> RC0402FR-071KL; Manufacturer (none) -> Yageo
- R12, R13, R8: MPN (none) -> RC0402FR-075K1L; Manufacturer (none) -> Yageo
- R16, R17, R24: MPN (none) -> RC0402FR-07100KL; Manufacturer (none) -> Yageo
- R20: MPN (none) -> RC0402FR-074K7L; Manufacturer (none) -> Yageo
- R23: MPN (none) -> RC0402FR-07732KL; Manufacturer (none) -> Yageo
- R25, R26, R28, R29: CircuitReference (none) -> https://www.ti.com/lit/ds/symlink/bq2970.pdf; Manufacturer (none) -> Yageo

Commit message: Apply selected non-boost capacitor identities without changing values
Fill23 missing MPNs and confirm3; retain clock revision, all geometry/copper and outstanding land/process gates.

Co-authored-by: Copilot <223556219+Copilot@users.noreply.github.com>
Parts:
- C1, C19, C20, C4, C5: MPN (none) -> GRM21BR61C106KE15L; Manufacturer (none) -> Murata
- C10, C11, C15, C17, C8: MPN (none) -> GRM155R61E105KA12D; Manufacturer (none) -> Murata
- C12, C13, C14, C16, C18, C23, C24, C6, C7, C9: MPN (none) -> GRM155R71C104KA88D; Manufacturer (none) -> Murata
- C21, C22: MPN (none) -> GRM1555C1H221JA01D; Manufacturer (none) -> Murata
- C25: MPN (none) -> GRM155R71C103KA01D; Manufacturer (none) -> Murata
- C30: CircuitReference (none) -> https://www.ti.com/lit/ds/symlink/bq2970.pdf; Manufacturer (none) -> Murata

Commit message: Correct USB slots and lands with local VBUS and CC route repairs
Restore source-bound slot geometry and secondary-anchor process; preserve 57 remaining opens and protected returns with zero native DRC errors.

Co-authored-by: Copilot <223556219+Copilot@users.noreply.github.com>
Parts:
- X6: footprint Adafruit Feather RP2040 Prop-Maker-import-fps:USB_C_CUSB31-CFM2AX-01-X -> Handbell:USB_C_HRO_TYPE_C_31_M_12_Handbell; MPN (none) -> TYPE-C-31-M-12; Manufacturer (none) -> HRO / Korean Hroparts Elec
Changed lines of the file:
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@@
 			)
 		)
-		(property "Footprint" "Adafruit Feather RP2040 Prop-Maker-import-fps:USB_C_CUSB31-CFM2AX-01-X"
+		(property "Footprint" "Handbell:USB_C_HRO_TYPE_C_31_M_12_Handbell"
 			(at 185.42 104.14 0)
 			(hide yes)
@@
 			)
 		)
-		(property "Datasheet" ""
+		(property "Datasheet" "https://jlcpcb.com/partdetail/Korean_HropartsElec-TYPE_C_31_M12/C165948"
 			(at 185.42 104.14 0)
 			(hide yes)
@@
 			)
 		)
-		(property "Description" ""
+		(property "Description" "HRO TYPE-C-31-M-12; modified slots/outer lands; secondary solder all four anchors."
 			(at 185.42 104.14 0)
 			(hide yes)
@@
 			)
 		)
+(property "MPN" "TYPE-C-31-M-12" (at 185.42 104.14 0)  (hide yes) (effects (font (size 1 1))))
+(property "Manufacturer" "HRO / Korean Hroparts Elec" (at 185.42 104.14 0)  (hide yes) (effects (font (size 1 1))))
 	)
 	(symbol

Commit message: Complete all 83 native part identities in one geometry-preserving batch
Apply the remaining 17 selected device and power identities; retain source geometry and publish one complete-identity schematic view.

Co-authored-by: Copilot <223556219+Copilot@users.noreply.github.com>
Parts:
- C26, C27, C28: MPN (none) -> GRM21BR61C226ME44L; Manufacturer (none) -> Murata
- CHG0: MPN (none) -> APT1608LSECK/J4-PRV; Manufacturer (none) -> Kingbright
- D3: MPN (none) -> 1N4148WS-7-F; Manufacturer (none) -> Diodes Incorporated
- D4: MPN (none) -> PMEG2020AEA,115; Manufacturer (none) -> Nexperia
- FB1, FB2: MPN (none) -> BLM18SG121TN1D; Manufacturer (none) -> Murata
- IC1: MPN (none) -> RP2040; Manufacturer (none) -> Raspberry Pi
- IC4: MPN (none) -> LSM6DSOXTR; Manufacturer (none) -> STMicroelectronics
- L0: MPN (none) -> APT1608LSECK/J3-PRV; Manufacturer (none) -> Kingbright
- L1: value 1uH (MPN pending) -> 1uH; MPN (none) -> VLS5045EX-1R0N; Manufacturer (none) -> TDK
- Q1: MPN (none) -> AO3401; Manufacturer (none) -> Alpha & Omega Semiconductor
- Q2: value C20917 -> AO3400A; MPN (none) -> AO3400A; Manufacturer (none) -> Alpha & Omega Semiconductor
- U2: MPN (none) -> RT9080-33GJ5; Manufacturer (none) -> Richtek
- U3: MPN (none) -> MCP73831T-2ACI/OT; Manufacturer (none) -> Microchip Technology
- U4: MPN (none) -> MAX98357AETE+T; Manufacturer (none) -> Analog Devices / Maxim Integrated
Changed lines of the file:
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@@
 			)
 		)
-		(property "Datasheet" ""
+		(property "Datasheet" "https://www.kingbrightusa.com/images/catalog/SPEC/APT1608LSECK-J4-PRV.pdf"
 			(at 162.56 50.8 0)
 			(hide yes)
@@
 			)
 		)
+(property "MPN" "APT1608LSECK/J4-PRV" (at 162.56 50.8 0)  (hide yes) (effects (font (size 1 1))))
+(property "Manufacturer" "Kingbright" (at 162.56 50.8 0)  (hide yes) (effects (font (size 1 1))))
 	)
 	(symbol
@@
 			)
 		)
-		(property "Datasheet" ""
+		(property "Datasheet" "https://www.kingbrightusa.com/images/catalog/SPEC/APT1608LSECK-J3-PRV.pdf"
 			(at 144.78 63.5 0)
 			(hide yes)
@@
 			)
 		)
+(property "MPN" "APT1608LSECK/J3-PRV" (at 144.78 63.5 0)  (hide yes) (effects (font (size 1 1))))
+(property "Manufacturer" "Kingbright" (at 144.78 63.5 0)  (hide yes) (effects (font (size 1 1))))
 	)
 	(symbol
@@
 			)
 		)
-		(property "Datasheet" ""
+		(property "Datasheet" "https://pim.murata.com/asset/pim4/ferriteBeadInductortypefilter/ENFA0003_PDF_FERRITEBEADINDUCTORTYPEFILTER?lastModifiedDatetime=20260603144239"
 			(at 347.98 170.18 0)
 			(hide yes)
@@
 			)
 		)
+(property "MPN" "BLM18SG121TN1D" (at 347.98 170.18 0)  (hide yes) (effects (font (size 1 1))))
+(property "Manufacturer" "Murata" (at 347.98 170.18 0)  (hide yes) (effects (font (size 1 1))))
 	)
 	(symbol
@@
 			)
 		)
-		(property "Datasheet" ""
+		(property "Datasheet" "https://www.aosmd.com/sites/default/files/res/datasheets/AO3401.pdf"
 			(at 284.48 218.44 0)
 			(hide yes)
@@
 			)
 		)
+(property "MPN" "AO3401" (at 284.48 218.44 0)  (hide yes) (effects (font (size 1 1))))
+(property "Manufacturer" "Alpha & Omega Semiconductor" (at 284.48 218.44 0)  (hide yes) (effects (font (size 1 1))))
 	)
 	(symbol
@@
 			)
 		)
-		(property "Datasheet" ""
+		(property "Datasheet" "https://www.richtek.com/assets/product_file/RT9080/DS9080-09.pdf"
 			(at 73.66 53.34 0)
 			(hide yes)
@@
 			)
 		)
+(property "MPN" "RT9080-33GJ5" (at 73.66 53.34 0)  (hide yes) (effects (font (size 1 1))))
+(property "Manufacturer" "Richtek" (at 73.66 53.34 0)  (hide yes) (effects (font (size 1 1))))
 	)
 	(symbol
@@
 			)
 		)
-		(property "Value" "C20917"
+		(property "Value" "AO3400A"
 			(at 279.4 237.49 0)
 			(show_name no)
@@
 			)
 		)
-		(property "Datasheet" ""
+		(property "Datasheet" "https://www.aosmd.com/sites/default/files/res/datasheets/AO3400A.pdf"
 			(at 284.48 236.22 0)
 			(hide yes)
@@
 			)
 		)
+(property "MPN" "AO3400A" (at 284.48 236.22 0)  (hide yes) (effects (font (size 1 1))))
+(property "Manufacturer" "Alpha & Omega Semiconductor" (at 284.48 236.22 0)  (hide yes) (effects (font (size 1 1))))
 	)
 	(symbol
@@
 			)
 		)
-		(property "Datasheet" ""
+		(property "Datasheet" "https://pim.murata.com/asset/pim4/ferriteBeadInductortypefilter/ENFA0003_PDF_FERRITEBEADINDUCTORTYPEFILTER?lastModifiedDatetime=20260603144239"
 			(at 347.98 162.56 0)
 			(hide yes)
@@
 			)
 		)
+(property "MPN" "BLM18SG121TN1D" (at 347.98 162.56 0)  (hide yes) (effects (font (size 1 1))))
+(property "Manufacturer" "Murata" (at 347.98 162.56 0)  (hide yes) (effects (font (size 1 1))))
 	)
 	(symbol
@@
 			)
 		)
-		(property "Datasheet" ""
+		(property "Datasheet" "https://www.diodes.com/datasheet/download/1N4148WS.pdf"
 			(at 114.3 43.18 0)
 			(hide yes)
@@
 			)
 		)
+(property "MPN" "1N4148WS-7-F" (at 114.3 43.18 0)  (hide yes) (effects (font (size 1 1))))
+(property "Manufacturer" "Diodes Incorporated" (at 114.3 43.18 0)  (hide yes) (effects (font (size 1 1))))
 	)
 	(symbol
@@
 			)
 		)
-		(property "Datasheet" ""
+		(property "Datasheet" "https://datasheets.raspberrypi.com/rp2040/rp2040-datasheet.pdf"
 			(at 93.98 190.5 0)
 			(hide yes)
@@
 			)
 		)
+(property "MPN" "RP2040" (at 93.98 190.5 0)  (hide yes) (effects (font (size 1 1))))
+(property "Manufacturer" "Raspberry Pi" (at 93.98 190.5 0)  (hide yes) (effects (font (size 1 1))))
 	)
 	(symbol
@@
 			)
 		)
-		(property "Datasheet" ""
+		(property "Datasheet" "https://ww1.microchip.com/downloads/aemDocuments/documents/APID/ProductDocuments/DataSheets/MCP73831-Family-Data-Sheet-DS20001984H.pdf"
 			(at 190.5 53.34 0)
 			(hide yes)
@@
 			)
 		)
+(property "MPN" "MCP73831T-2ACI/OT" (at 190.5 53.34 0)  (hide yes) (effects (font (size 1 1))))
+(property "Manufacturer" "Microchip Technology" (at 190.5 53.34 0)  (hide yes) (effects (font (size 1 1))))
 	)
 	(symbol
@@
 			)
 		)
-		(property "Datasheet" ""
+		(property "Datasheet" "https://cdn-shop.adafruit.com/product-files/3006/MAX98357A-MAX98357B.pdf"
 			(at 327.66 170.18 0)
 			(hide yes)
@@
 			)
 		)
+(property "MPN" "MAX98357AETE+T" (at 327.66 170.18 0)  (hide yes) (effects (font (size 1 1))))
+(property "Manufacturer" "Analog Devices / Maxim Integrated" (at 327.66 170.18 0)  (hide yes) (effects (font (size 1 1))))
 	)
 	(symbol
@@
 			)
 		)
-		(property "Datasheet" ""
+		(property "Datasheet" "https://assets.nexperia.com/documents/data-sheet/PMEG2020AEA.pdf"
 			(at 38.1 50.8 0)
 			(hide yes)
@@
 			)
 		)
+(property "MPN" "PMEG2020AEA,115" (at 38.1 50.8 0)  (hide yes) (effects (font (size 1 1))))
+(property "Manufacturer" "Nexperia" (at 38.1 50.8 0)  (hide yes) (effects (font (size 1 1))))
 	)
 	(symbol
@@
 			)
 		)
-		(property "Datasheet" ""
+		(property "Datasheet" "https://datasheet.lcsc.com/datasheet/pdf/fa6a99ef5791a87a2f52fed9abb2f6b1.pdf?productCode=C481766"
 			(at 208.2800 195.5800 0)
 			(hide yes)
@@
 		)
 		(instances (project "handbell" (path "/85874120-e238-4c38-82e5-c93e2e8375b3" (reference "IC4") (unit 1))))
+(property "MPN" "LSM6DSOXTR" (at 208.2800 195.5800 0)  (hide yes) (effects (font (size 1 1))))
+(property "Manufacturer" "STMicroelectronics" (at 208.2800 195.5800 0)  (hide yes) (effects (font (size 1 1))))
 	)
 (symbol
@@
 			)
 		)
-		(property "Value" "1uH (MPN pending)"
+		(property "Value" "1uH"
 			(at 335.28 65.04 0)
 			(show_name no)
@@
 			)
 		)
-		(property "Datasheet" ""
+		(property "Datasheet" "https://product.tdk.com/en/search/inductor/inductor/smd/info?part_no=VLS5045EX-1R0N"
 			(at 335.28 63.5 0)
 			(hide yes)
@@
 			)
 		)
+(property "MPN" "VLS5045EX-1R0N" (at 335.28 63.5 0)  (hide yes) (effects (font (size 1 1))))
+(property "Manufacturer" "TDK" (at 335.28 63.5 0)  (hide yes) (effects (font (size 1 1))))
 	)
 (symbol
@@
 			)
 		)
-		(property "Datasheet" ""
+		(property "Datasheet" "https://pim.murata.com/asset/pim4/ceramicCapacitorSMD/GRM21BR61C226ME44-01A-EN_PDF_CERAMICCAPACITORSMD?lastModifiedDatetime=20260730170906"
 			(at 304.8 88.9 0)
 			(hide yes)
@@
 			)
 		)
+(property "MPN" "GRM21BR61C226ME44L" (at 304.8 88.9 0)  (hide yes) (effects (font (size 1 1))))
+(property "Manufacturer" "Murata" (at 304.8 88.9 0)  (hide yes) (effects (font (size 1 1))))
 	)
 (symbol
@@
 			)
 		)
-		(property "Datasheet" ""
+		(property "Datasheet" "https://pim.murata.com/asset/pim4/ceramicCapacitorSMD/GRM21BR61C226ME44-01A-EN_PDF_CERAMICCAPACITORSMD?lastModifiedDatetime=20260730170906"
 			(at 375.92 88.9 0)
 			(hide yes)
@@
 			)
 		)
+(property "MPN" "GRM21BR61C226ME44L" (at 375.92 88.9 0)  (hide yes) (effects (font (size 1 1))))
+(property "Manufacturer" "Murata" (at 375.92 88.9 0)  (hide yes) (effects (font (size 1 1))))
 	)
 (symbol
@@
 			)
 		)
-		(property "Datasheet" ""
+		(property "Datasheet" "https://pim.murata.com/asset/pim4/ceramicCapacitorSMD/GRM21BR61C226ME44-01A-EN_PDF_CERAMICCAPACITORSMD?lastModifiedDatetime=20260730170906"
 			(at 388.62 88.9 0)
 			(hide yes)
@@
 			)
 		)
+(property "MPN" "GRM21BR61C226ME44L" (at 388.62 88.9 0)  (hide yes) (effects (font (size 1 1))))
+(property "Manufacturer" "Murata" (at 388.62 88.9 0)  (hide yes) (effects (font (size 1 1))))
 	)
 (symbol

Commit message: Land selected power footprints and publish standalone ground checks
Preserve existing copper and quiet pickoffs across eleven land revisions. Publish the source-bound 56-open checkpoint, reusable fill plan/checker, and owner-requested pause handoff.

Co-authored-by: Copilot <223556219+Copilot@users.noreply.github.com>
Parts:
- C1, C19, C20, C4, C5: footprint Adafruit Feather RP2040 Prop-Maker-import-fps:0805-NO -> Handbell:Murata_GRM21_10uF_Reflow
- C26, C27, C28: footprint Adafruit Feather RP2040 Prop-Maker-import-fps:0805-NO -> Handbell:Murata_GRM21_22uF_Reflow
- FB1, FB2: footprint Adafruit Feather RP2040 Prop-Maker-import-fps:0603-NO -> Handbell:Murata_BLM18SG121_WideCopper
- L1: footprint Adafruit TPS61023-import-fps:INDUCTOR_5X5MM_TDK_VLC5045 -> Handbell:TDK_VLS5045EX_Reflow
Changed lines of the file:
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@@
 			)
 		)
-		(property "Footprint" "Adafruit Feather RP2040 Prop-Maker-import-fps:0805-NO"
+		(property "Footprint" "Handbell:Murata_GRM21_10uF_Reflow"
 			(at 86.36 63.5 0)
 			(hide yes)
@@
 			)
 		)
-		(property "Footprint" "Adafruit Feather RP2040 Prop-Maker-import-fps:0603-NO"
+		(property "Footprint" "Handbell:Murata_BLM18SG121_WideCopper"
 			(at 347.98 170.18 0)
 			(hide yes)
@@
 			)
 		)
-		(property "Footprint" "Adafruit Feather RP2040 Prop-Maker-import-fps:0603-NO"
+		(property "Footprint" "Handbell:Murata_BLM18SG121_WideCopper"
 			(at 347.98 162.56 0)
 			(hide yes)
@@
 			)
 		)
-		(property "Footprint" "Adafruit Feather RP2040 Prop-Maker-import-fps:0805-NO"
+		(property "Footprint" "Handbell:Murata_GRM21_10uF_Reflow"
 			(at 93.98 63.5 0)
 			(hide yes)
@@
 			)
 		)
-		(property "Footprint" "Adafruit Feather RP2040 Prop-Maker-import-fps:0805-NO"
+		(property "Footprint" "Handbell:Murata_GRM21_10uF_Reflow"
 			(at 218.44 58.42 0)
 			(hide yes)
@@
 			)
 		)
-		(property "Footprint" "Adafruit Feather RP2040 Prop-Maker-import-fps:0805-NO"
+		(property "Footprint" "Handbell:Murata_GRM21_10uF_Reflow"
 			(at 294.64 182.88 0)
 			(hide yes)
@@
 			)
 		)
-		(property "Footprint" "Adafruit Feather RP2040 Prop-Maker-import-fps:0805-NO"
+		(property "Footprint" "Handbell:Murata_GRM21_10uF_Reflow"
 			(at 48.26 63.5 0)
 			(hide yes)
@@
 			)
 		)
-		(property "Footprint" "Adafruit TPS61023-import-fps:INDUCTOR_5X5MM_TDK_VLC5045"
+		(property "Footprint" "Handbell:TDK_VLS5045EX_Reflow"
 			(at 335.28 63.5 0)
 			(hide yes)
@@
 			)
 		)
-		(property "Footprint" "Adafruit Feather RP2040 Prop-Maker-import-fps:0805-NO"
+		(property "Footprint" "Handbell:Murata_GRM21_22uF_Reflow"
 			(at 304.8 88.9 0)
 			(hide yes)
@@
 			)
 		)
-		(property "Footprint" "Adafruit Feather RP2040 Prop-Maker-import-fps:0805-NO"
+		(property "Footprint" "Handbell:Murata_GRM21_22uF_Reflow"
 			(at 375.92 88.9 0)
 			(hide yes)
@@
 			)
 		)
-		(property "Footprint" "Adafruit Feather RP2040 Prop-Maker-import-fps:0805-NO"
+		(property "Footprint" "Handbell:Murata_GRM21_22uF_Reflow"
 			(at 388.62 88.9 0)
 			(hide yes)

Commit message: Close boost and shunt lands with bounded local repairs
Apply recorded U5/R27 patterns and envelopes. Preserve trace widths and fixed poses; enlarge the R27.2 exclusion with its land. Reuse unaffected primitive evidence and bind the final filled continuity proof.

Co-authored-by: Copilot <223556219+Copilot@users.noreply.github.com>
Parts:
- R27: footprint T8:ERJ6BW_0805 -> Handbell:ERJ6BW_0805_Panasonic_Example
- U5: footprint Adafruit TPS61023-import-fps:SOT563 -> Handbell:TPS61023_DRL_TI_Example
Changed lines of the file:
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@@
 			)
 		)
-		(property "Footprint" "Adafruit TPS61023-import-fps:SOT563"
+		(property "Footprint" "Handbell:TPS61023_DRL_TI_Example"
 			(at 335.28 91.44 0)
 			(hide yes)
@@
 (wire (pts (xy 256.54 342.9) (xy 261.62 342.9)) (stroke (width 0) (type default)))
 (label "PROT_COUT"  (at 261.62 342.9 0) (effects (font (size 1.016 1.016)) (justify left bottom)))
-(symbol (lib_id "T8:R") (at 317.5 350.52 0) (unit 1) (in_bom yes) (on_board yes) (dnp no) (property "Reference" "R27" (at 317.5 346.71 0)  (effects (font (size 1.016 1.016)))) (property "Value" "33m 1% 0.5W" (at 317.5 354.33 0)  (effects (font (size 1.016 1.016)))) (property "Footprint" "T8:ERJ6BW_0805" (at 317.5 350.52 0) (hide yes) (effects (font (size 1.016 1.016)))) (property "Datasheet" "https://industrial.panasonic.com/ww/products/pt/thick-film-chip-resistors" (at 317.5 350.52 0) (hide yes) (effects (font (size 1.016 1.016)))) (property "MPN" "ERJ-6BWFR033V" (at 317.5 350.52 0) (hide yes) (effects (font (size 1.016 1.016)))) (pin "1")(pin "2") (instances (project "handbell" (path "/85874120-e238-4c38-82e5-c93e2e8375b3" (reference "R27") (unit 1)))))
+(symbol (lib_id "T8:R") (at 317.5 350.52 0) (unit 1) (in_bom yes) (on_board yes) (dnp no) (property "Reference" "R27" (at 317.5 346.71 0)  (effects (font (size 1.016 1.016)))) (property "Value" "33m 1% 0.5W" (at 317.5 354.33 0)  (effects (font (size 1.016 1.016)))) (property "Footprint" "Handbell:ERJ6BW_0805_Panasonic_Example" (at 317.5 350.52 0) (hide yes) (effects (font (size 1.016 1.016)))) (property "Datasheet" "https://industrial.panasonic.com/ww/products/pt/thick-film-chip-resistors" (at 317.5 350.52 0) (hide yes) (effects (font (size 1.016 1.016)))) (property "MPN" "ERJ-6BWFR033V" (at 317.5 350.52 0) (hide yes) (effects (font (size 1.016 1.016)))) (pin "1")(pin "2") (instances (project "handbell" (path "/85874120-e238-4c38-82e5-c93e2e8375b3" (reference "R27") (unit 1)))))
 (wire (pts (xy 312.42 350.52) (xy 307.34 350.52)) (stroke (width 0) (type default)))
 (label "PROT_FET_RETURN"  (at 307.34 350.52 0) (effects (font (size 1.016 1.016)) (justify right bottom)))
