File: hardware/handbell/iterations/printed-bell-clock-draft/handbell.kicad_pcb (KiCad board)
At the start: 2 copper layers, 44.5 x 48.3 mm, 104 parts, among them IC1 RP2040_QFN56, IC4 LSM6DSOXTR, J1 504050-0291, J2 SM02B-SRSS-TB, Q1 AO3401, Q2 AO3400A, Q3 DMP2045UFY4, Q4 AO3400A, Q5 CSD83325L, U1 W25Q16JVUXIQ TR / 2MB, U2 RT9080-3.3, U3 MCP73831T-2ACI/OT, U4 MAX98357A, U5 TPS61023DRLR, U6 BQ29700DSER, X6 USB Type C, Y1 12MHz/CL10pF

Commit message: Free the MCU power corridor and connect the regulator output
Retain all nine ground vias in a staggered array and move the unchanged-width VHI feed through the central B neck. Reuse the C8 experiment, preserve contact exclusions and prior connectivity, and record thermal/stencil limits.

Co-authored-by: Copilot <223556219+Copilot@users.noreply.github.com>
Routing:
- net VHI: track 64.6 -> 60.6 mm
- net GND: track 115.7 -> 114.1 mm
- net VCORE: track 6.12 -> 7.70 mm
Changed lines of the file:
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@@
 (segment (start 104.991300 100.898100) (end 104.991000 100.898000) (width 0.1778) (layer "F.Cu") (net "+3V3"))
 (segment (start 103.450000 102.600000) (end 103.550000 102.700000) (width 0.1778) (layer "F.Cu") (net "+3V3"))
-(segment (start 104.178100 102.450100) (end 104.178100 102.200000) (width 0.1778) (layer "F.Cu") (net "+3V3"))
 (segment (start 103.928200 102.700000) (end 104.178100 102.450100) (width 0.1778) (layer "F.Cu") (net "+3V3"))
 (segment (start 103.550000 102.700000) (end 103.928200 102.700000) (width 0.1778) (layer "F.Cu") (net "+3V3"))
@@
 (segment (start 95.312300 102.304500) (end 95.312100 102.304700) (width 0.1778) (layer "F.Cu") (net "+3V3"))
 (segment (start 95.312100 102.304900) (end 95.312300 102.305000) (width 0.1778) (layer "F.Cu") (net "+3V3"))
-(segment (start 103.450000 102.200000) (end 104.050000 102.200000) (width 0.1778) (layer "F.Cu") (net "+3V3"))
-(segment (start 104.200000 101.700000) (end 105.000000 100.900000) (width 0.1778) (layer "F.Cu") (net "+3V3"))
-(segment (start 104.200000 102.050000) (end 104.200000 101.700000) (width 0.1778) (layer "F.Cu") (net "+3V3"))
-(segment (start 104.050000 102.200000) (end 104.200000 102.050000) (width 0.1778) (layer "F.Cu") (net "+3V3"))
-(segment (start 104.050000 102.200000) (end 104.178100 102.200000) (width 0.1778) (layer "F.Cu") (net "+3V3"))
+(segment (start 103.450000 102.200000) (end 103.9 102.2) (width 0.1778) (layer "F.Cu") (net "+3V3"))
 (segment (start 103.550000 102.700000) (end 104.050000 103.200000) (width 0.1778) (layer "F.Cu") (net "+3V3"))
 (segment (start 102.999200 107.011500) (end 102.999200 106.420900) (width 0.1778) (layer "F.Cu") (net "+3V3"))
@@
 (segment (start 91.992000 104.200000) (end 97.500000 104.200000) (width 0.1778) (layer "F.Cu") (net "VBAT"))
 (segment (start 91.992000 105.300000) (end 91.992000 104.200000) (width 0.1778) (layer "F.Cu") (net "VBAT"))
-(segment (start 99.200000 99.200000) (end 100.000000 99.200000) (width 0.6) (layer "B.Cu") (net "GND"))
-(segment (start 99.200000 99.200000) (end 99.200000 100.000000) (width 0.6) (layer "B.Cu") (net "GND"))
-(segment (start 99.200000 100.000000) (end 100.000000 100.000000) (width 0.6) (layer "B.Cu") (net "GND"))
-(segment (start 99.200000 100.000000) (end 99.200000 100.800000) (width 0.6) (layer "B.Cu") (net "GND"))
-(segment (start 99.200000 100.800000) (end 100.000000 100.800000) (width 0.6) (layer "B.Cu") (net "GND"))
-(segment (start 100.000000 99.200000) (end 100.800000 99.200000) (width 0.6) (layer "B.Cu") (net "GND"))
-(segment (start 100.000000 99.200000) (end 100.000000 100.000000) (width 0.6) (layer "B.Cu") (net "GND"))
-(segment (start 100.000000 100.000000) (end 100.800000 100.000000) (width 0.6) (layer "B.Cu") (net "GND"))
-(segment (start 100.000000 100.000000) (end 100.000000 100.800000) (width 0.6) (layer "B.Cu") (net "GND"))
-(segment (start 100.000000 100.800000) (end 100.800000 100.800000) (width 0.6) (layer "B.Cu") (net "GND"))
-(segment (start 100.800000 99.200000) (end 100.800000 100.000000) (width 0.6) (layer "B.Cu") (net "GND"))
-(segment (start 100.800000 100.000000) (end 100.800000 100.800000) (width 0.6) (layer "B.Cu") (net "GND"))
+(segment (start 99.15 99.38) (end 99.8 99.07) (width 0.6) (layer "B.Cu") (net "GND"))
+(segment (start 99.15 101.24) (end 99.8 100.93) (width 0.6) (layer "B.Cu") (net "GND"))
+(segment (start 99.15 98.76) (end 99.8 99.07) (width 0.6) (layer "B.Cu") (net "GND"))
+(segment (start 99.8 99.69) (end 99.8 100.31) (width 0.6) (layer "B.Cu") (net "GND"))
+(segment (start 99.8 100.31) (end 99.8 100.93) (width 0.6) (layer "B.Cu") (net "GND"))
+(segment (start 99.15 100.0) (end 99.15 100.62) (width 0.6) (layer "B.Cu") (net "GND"))
+(segment (start 99.8 99.07) (end 99.8 99.69) (width 0.6) (layer "B.Cu") (net "GND"))
+(segment (start 99.15 99.38) (end 99.15 100.0) (width 0.6) (layer "B.Cu") (net "GND"))
+(segment (start 99.15 100.62) (end 99.15 101.24) (width 0.6) (layer "B.Cu") (net "GND"))
+(segment (start 99.15 100.62) (end 99.8 100.31) (width 0.6) (layer "B.Cu") (net "GND"))
+(segment (start 99.15 100.0) (end 99.8 99.69) (width 0.6) (layer "B.Cu") (net "GND"))
+(segment (start 99.15 98.76) (end 99.15 99.38) (width 0.6) (layer "B.Cu") (net "GND"))
 (segment (start 110.400323 89.587211) (end 111.050323 89.587211) (width 0.6) (layer "B.Cu") (net "GND"))
 (segment (start 110.400323 89.587211) (end 110.400323 90.237211) (width 0.6) (layer "B.Cu") (net "GND"))
@@
 (segment (start 92.600000 108.000000) (end 92.600000 109.300000) (width 1.2) (layer "F.Cu") (net "V+"))
 (segment (start 92.600000 109.300000) (end 91.450000 110.900000) (width 1.2) (layer "F.Cu") (net "V+"))
-(segment (start 100.000000 97.700000) (end 102.300000 97.700000) (width 0.8) (layer "F.Cu") (net "VHI"))
-(segment (start 102.300000 97.700000) (end 102.300000 102.300000) (width 0.8) (layer "F.Cu") (net "VHI"))
-(segment (start 102.300000 102.300000) (end 100.000000 102.300000) (width 0.8) (layer "F.Cu") (net "VHI"))
+(segment (start 100 97.7) (end 100.8 98.5) (width 0.8) (layer "B.Cu") (net "VHI"))
+(segment (start 100.8 98.5) (end 100.8 101.5) (width 0.8) (layer "B.Cu") (net "VHI"))
+(segment (start 100.8 101.5) (end 100 102.3) (width 0.8) (layer "B.Cu") (net "VHI"))
 (segment (start 95.100000 106.000000) (end 94.600000 107.050000) (width 0.8) (layer "F.Cu") (net "VHI"))
 (segment (start 98.999141 91.501032) (end 100.000000 92.500000) (width 0.8) (layer "F.Cu") (net "VHI"))
@@
 (segment (start 90.400000 94.500000) (end 90.412306 94.492711) (width 0.25) (layer "F.Cu") (net "+3V3"))
 (segment (start 104.991429 100.897675) (end 105.000000 100.900000) (width 0.25) (layer "F.Cu") (net "+3V3"))
-(segment (start 105.000000 100.900000) (end 104.400000 101.500000) (width 0.25) (layer "F.Cu") (net "+3V3"))
-(segment (start 104.400000 101.500000) (end 104.400000 101.700000) (width 0.25) (layer "F.Cu") (net "+3V3"))
-(segment (start 104.400000 101.700000) (end 104.350000 101.750000) (width 0.25) (layer "F.Cu") (net "+3V3"))
-(segment (start 104.350000 101.750000) (end 104.350000 105.150000) (width 0.25) (layer "F.Cu") (net "+3V3"))
+(segment (start 104.35 102.4) (end 104.350000 105.150000) (width 0.25) (layer "F.Cu") (net "+3V3"))
 (segment (start 104.350000 105.150000) (end 105.850000 106.650000) (width 0.25) (layer "F.Cu") (net "+3V3"))
 (segment (start 105.850000 106.650000) (end 105.900000 106.650000) (width 0.25) (layer "F.Cu") (net "+3V3"))
@@
 (via (at 101.802000 93.005500) (size 0.6) (drill 0.3) (layers "F.Cu" "B.Cu") (net "+3V3"))
 (via (at 106.095600 93.005500) (size 0.6) (drill 0.3) (layers "F.Cu" "B.Cu") (net "+3V3"))
-(via (at 99.200000 99.200000) (size 0.604) (drill 0.35) (layers "F.Cu" "B.Cu") (net "GND"))
-(via (at 99.200000 100.000000) (size 0.604) (drill 0.35) (layers "F.Cu" "B.Cu") (net "GND"))
-(via (at 99.200000 100.800000) (size 0.604) (drill 0.35) (layers "F.Cu" "B.Cu") (net "GND"))
-(via (at 100.000000 99.200000) (size 0.604) (drill 0.35) (layers "F.Cu" "B.Cu") (net "GND"))
-(via (at 100.000000 100.000000) (size 0.604) (drill 0.35) (layers "F.Cu" "B.Cu") (net "GND"))
-(via (at 100.000000 100.800000) (size 0.604) (drill 0.35) (layers "F.Cu" "B.Cu") (net "GND"))
-(via (at 100.800000 99.200000) (size 0.604) (drill 0.35) (layers "F.Cu" "B.Cu") (net "GND"))
-(via (at 100.800000 100.000000) (size 0.604) (drill 0.35) (layers "F.Cu" "B.Cu") (net "GND"))
-(via (at 100.800000 100.800000) (size 0.604) (drill 0.35) (layers "F.Cu" "B.Cu") (net "GND"))
+(via (at 99.15 98.76) (size 0.604) (drill 0.35) (layers "F.Cu" "B.Cu") (net "GND"))
+(via (at 99.15 99.38) (size 0.604) (drill 0.35) (layers "F.Cu" "B.Cu") (net "GND"))
+(via (at 99.15 100.0) (size 0.604) (drill 0.35) (layers "F.Cu" "B.Cu") (net "GND"))
+(via (at 99.15 100.62) (size 0.604) (drill 0.35) (layers "F.Cu" "B.Cu") (net "GND"))
+(via (at 99.15 101.24) (size 0.604) (drill 0.35) (layers "F.Cu" "B.Cu") (net "GND"))
+(via (at 99.8 99.07) (size 0.604) (drill 0.35) (layers "F.Cu" "B.Cu") (net "GND"))
+(via (at 99.8 99.69) (size 0.604) (drill 0.35) (layers "F.Cu" "B.Cu") (net "GND"))
+(via (at 99.8 100.31) (size 0.604) (drill 0.35) (layers "F.Cu" "B.Cu") (net "GND"))
+(via (at 99.8 100.93) (size 0.604) (drill 0.35) (layers "F.Cu" "B.Cu") (net "GND"))
 (via (at 110.400323 89.587211) (size 0.604) (drill 0.35) (layers "F.Cu" "B.Cu") (net "GND"))
 (via (at 110.400323 90.237211) (size 0.604) (drill 0.35) (layers "F.Cu" "B.Cu") (net "GND"))
@@
 (segment (start 103.45 99.8) (end 104.1 99.8) (width 0.2) (layer "F.Cu") (net "VCORE"))
 (segment (start 104.1 99.8) (end 104.299744 99.999744) (width 0.2) (layer "F.Cu") (net "VCORE"))
-(segment (start 104.299744 99.999744) (end 104.989898 99.999744) (width 0.2) (layer "F.Cu") (net "VCORE")))
+(segment (start 104.299744 99.999744) (end 104.989898 99.999744) (width 0.2) (layer "F.Cu") (net "VCORE"))
+(segment (start 103.45 100.2) (end 102.65 100.2) (width 0.2) (layer "F.Cu") (net "+3V3"))
+(segment (start 102.65 100.2) (end 102.65 102.2) (width 0.25) (layer "F.Cu") (net "+3V3"))
+(segment (start 102.65 102.2) (end 103.45 102.2) (width 0.2) (layer "F.Cu") (net "+3V3"))
+(segment (start 103.9 102.2) (end 104.1 102.4) (width 0.2) (layer "F.Cu") (net "+3V3"))
+(segment (start 104.1 102.4) (end 104.35 102.4) (width 0.2) (layer "F.Cu") (net "+3V3"))
+(segment (start 103.45 101.8) (end 104.1 101.8) (width 0.2) (layer "F.Cu") (net "VCORE"))
+(segment (start 104.1 101.8) (end 104.2 101.9) (width 0.2) (layer "F.Cu") (net "VCORE"))
+(segment (start 104.2 101.9) (end 104.9931 101.9) (width 0.2) (layer "F.Cu") (net "VCORE")))

Commit message: Connect the charge-indicator branch with preserved ground continuity
Accept seven 0.20 mm front tracks between R2 and CHG0. Preserve existing copper, parts, vias, schematic and private returns; 51 opens remain.

Co-authored-by: Copilot <223556219+Copilot@users.noreply.github.com>
Routing:
- net Net-(CHG0-PadC): track 0.00 -> 2.87 mm
Changed lines of the file:
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@@
 (segment (start 103.45 101.8) (end 104.1 101.8) (width 0.2) (layer "F.Cu") (net "VCORE"))
 (segment (start 104.1 101.8) (end 104.2 101.9) (width 0.2) (layer "F.Cu") (net "VCORE"))
-(segment (start 104.2 101.9) (end 104.9931 101.9) (width 0.2) (layer "F.Cu") (net "VCORE")))
+(segment (start 104.2 101.9) (end 104.9931 101.9) (width 0.2) (layer "F.Cu") (net "VCORE"))
+(segment (start 104.00705 81.295629) (end 104.0 81.3) (width 0.2) (layer "F.Cu") (net "Net-(CHG0-PadC)"))
+(segment (start 104.0 81.3) (end 104.4 81.7) (width 0.2) (layer "F.Cu") (net "Net-(CHG0-PadC)"))
+(segment (start 104.4 81.7) (end 104.4 81.75) (width 0.2) (layer "F.Cu") (net "Net-(CHG0-PadC)"))
+(segment (start 104.4 81.75) (end 104.55 81.9) (width 0.2) (layer "F.Cu") (net "Net-(CHG0-PadC)"))
+(segment (start 104.55 81.9) (end 106.3 81.9) (width 0.2) (layer "F.Cu") (net "Net-(CHG0-PadC)"))
+(segment (start 106.3 81.9) (end 106.5 82.1) (width 0.2) (layer "F.Cu") (net "Net-(CHG0-PadC)"))
+(segment (start 106.5 82.1) (end 106.499567 82.101987) (width 0.2) (layer "F.Cu") (net "Net-(CHG0-PadC)")))
