File: hardware/handbell/iterations/printed-bell-four-layer/reports/imu-coupled-working.kicad_pcb (KiCad board)
At the start: 4 copper layers, 44.5 x 48.3 mm, 104 parts, among them IC1 RP2040_QFN56, IC4 LSM6DSOXTR, J1 504050-0291, J2 SM02B-SRSS-TB, Q1 AO3401, Q2 AO3400A, Q3 DMP2045UFY4, Q4 AO3400A, Q5 CSD83325L, U1 W25Q16JVUXIQ TR / 2MB, U2 RT9080-3.3, U3 MCP73831T-2ACI/OT, U4 MAX98357A, U5 TPS61023DRLR, U6 BQ29700DSER, X6 USB Type C, Y1 12MHz/CL10pF

Commit message: Preserve staged IMU supply interrupt routing and source-bound review views
Co-authored-by: Copilot <223556219+Copilot@users.noreply.github.com>
Routing:
- net +3V3: track 149.7 -> 157.2 mm
- net /IMU_INT2: track 18.5 -> 24.5 mm, vias 2 -> 3
- net GND: track 118.9 -> 120.4 mm
Changed lines of the file:
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@@
 (via (at 90.700000 91.650000) (size 0.604) (drill 0.35) (layers "F.Cu" "B.Cu") (net "GND"))
 (segment (start 90.700000 91.650000) (end 90.249806 92.330211) (width 0.3000) (layer "F.Cu") (net "GND"))
+(segment (start 90.249806 92.330211) (end 89.749806 92.330211) (width 0.3000) (layer "F.Cu") (net "GND"))
+(segment (start 89.749806 92.330211) (end 89.249806 92.330211) (width 0.3000) (layer "F.Cu") (net "GND"))
+(segment (start 88.587306 93.492711) (end 88.587306 93.992711) (width 0.3000) (layer "F.Cu") (net "GND"))
+(segment (start 88.749806 94.655211) (end 88.749806 95.250000) (width 0.2500) (layer "F.Cu") (net "+3V3"))
+(segment (start 88.749806 95.250000) (end 91.261752 95.250000) (width 0.2500) (layer "F.Cu") (net "+3V3"))
+(segment (start 91.261752 95.250000) (end 92.004083 94.507669) (width 0.2500) (layer "F.Cu") (net "+3V3"))
+(segment (start 92.004083 94.507669) (end 92.850000 94.000000) (width 0.2500) (layer "F.Cu") (net "+3V3"))
+(segment (start 92.850000 94.000000) (end 92.850000 93.350000) (width 0.2500) (layer "F.Cu") (net "+3V3"))
+(segment (start 92.004083 94.507669) (end 91.450000 94.200000) (width 0.2500) (layer "F.Cu") (net "+3V3"))
+(segment (start 91.450000 94.200000) (end 90.412306 93.992711) (width 0.2500) (layer "F.Cu") (net "+3V3"))
+(segment (start 89.249806 94.655211) (end 89.249806 94.250000) (width 0.1778) (layer "F.Cu") (net "/IMU_INT2"))
+(segment (start 89.249806 94.250000) (end 89.619500 93.580900) (width 0.1778) (layer "F.Cu") (net "/IMU_INT2"))
+(segment (start 89.619500 93.580900) (end 90.800000 92.750000) (width 0.1778) (layer "In2.Cu") (net "/IMU_INT2"))
+(segment (start 90.800000 92.750000) (end 93.100000 92.750000) (width 0.1778) (layer "In2.Cu") (net "/IMU_INT2"))
+(segment (start 93.100000 92.750000) (end 94.040000 92.310200) (width 0.1778) (layer "In2.Cu") (net "/IMU_INT2"))
+(via (at 89.619500 93.580900) (size 0.604) (drill 0.35) (layers "F.Cu" "B.Cu") (net "/IMU_INT2"))
 )

Commit message: Preserve repaired supply tree and release coupled IMU signal plan
Co-authored-by: Copilot <223556219+Copilot@users.noreply.github.com>
Routing:
- net +3V3: track 157.2 -> 170.6 mm, vias 12 -> 14
Changed lines of the file:
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@@
 (segment (start 93.100000 92.750000) (end 94.040000 92.310200) (width 0.1778) (layer "In2.Cu") (net "/IMU_INT2"))
 (via (at 89.619500 93.580900) (size 0.604) (drill 0.35) (layers "F.Cu" "B.Cu") (net "/IMU_INT2"))
+(via (at 87.850000 92.700000) (size 0.604) (drill 0.35) (layers "F.Cu" "B.Cu") (net "+3V3"))
+(segment (start 88.587306 92.992711) (end 87.850000 92.700000) (width 0.2500) (layer "F.Cu") (net "+3V3"))
+(via (at 88.150000 91.800000) (size 0.604) (drill 0.35) (layers "F.Cu" "B.Cu") (net "+3V3"))
+(segment (start 88.794835 91.491614) (end 88.150000 91.800000) (width 0.1778) (layer "F.Cu") (net "+3V3"))
+(segment (start 87.094469 95.226030) (end 88.000000 95.226030) (width 0.1778) (layer "F.Cu") (net "+3V3"))
+(segment (start 88.000000 95.226030) (end 88.749806 95.250000) (width 0.1778) (layer "F.Cu") (net "+3V3"))
+(segment (start 87.082668 93.109941) (end 87.850000 92.700000) (width 0.1778) (layer "F.Cu") (net "+3V3"))
+(segment (start 86.600000 93.109900) (end 87.082668 93.109941) (width 0.1778) (layer "F.Cu") (net "+3V3"))
+(segment (start 88.393800 90.500000) (end 88.794835 91.491614) (width 0.1778) (layer "F.Cu") (net "+3V3"))
+(segment (start 87.850000 92.700000) (end 88.200000 92.900000) (width 0.4000) (layer "In2.Cu") (net "+3V3"))
+(segment (start 88.150000 91.800000) (end 88.200000 92.900000) (width 0.4000) (layer "In2.Cu") (net "+3V3"))
+(segment (start 88.200000 92.900000) (end 88.600000 93.200000) (width 0.4000) (layer "In2.Cu") (net "+3V3"))
+(segment (start 88.600000 93.200000) (end 88.700000 94.300000) (width 0.4000) (layer "In2.Cu") (net "+3V3"))
+(segment (start 88.700000 94.300000) (end 90.000000 94.300000) (width 0.4000) (layer "In2.Cu") (net "+3V3"))
+(segment (start 90.000000 94.300000) (end 92.400000 94.200000) (width 0.4000) (layer "In2.Cu") (net "+3V3"))
+(segment (start 92.400000 94.200000) (end 92.800000 93.600000) (width 0.4000) (layer "In2.Cu") (net "+3V3"))
+(segment (start 92.800000 93.600000) (end 92.850000 93.350000) (width 0.4000) (layer "In2.Cu") (net "+3V3"))
 )

Commit message: Preserve complete local IMU primitive routing for electrical qualification
Co-authored-by: Copilot <223556219+Copilot@users.noreply.github.com>
Parts:
- moved R15 0.50 mm to (87.1, 92.1)
Routing:
- net SDA: track 13.3 -> 25.3 mm, vias 1 -> 3
- net INT: track 0.00 -> 6.91 mm, vias 0 -> 2
- net SCL: track 13.9 -> 19.1 mm, vias 0 -> 2
- net +3V3: track 170.6 -> 173.2 mm
- net GND: track 120.4 -> 120.5 mm, vias 26 -> 25
Changed lines of the file:
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@@
 (net "SDA"))
 	(embedded_fonts no)
-(at 87.082668 92.601941 90)
+(at 87.082668 92.101941 90)
 (property "MPN" "RC0402FR-0710KL" (at 0 0 0) (layer "F.Fab") (hide yes) (effects (font (size 1 1))))
 (property "Manufacturer" "Yageo" (at 0 0 0) (layer "F.Fab") (hide yes) (effects (font (size 1 1)))))
@@
 (segment (start 86.396500 93.018400) (end 85.013200 94.401700) (width 0.1778) (layer "F.Cu") (net "+3V3"))
 (segment (start 86.402100 93.018400) (end 86.396500 93.018400) (width 0.1778) (layer "F.Cu") (net "+3V3"))
-(segment (start 86.600000 91.540700) (end 86.402100 91.738600) (width 0.1778) (layer "F.Cu") (net "+3V3"))
 (segment (start 86.402100 93.018400) (end 86.402100 91.738600) (width 0.1778) (layer "F.Cu") (net "+3V3"))
 (segment (start 106.310600 92.790500) (end 106.095600 93.005500) (width 0.1778) (layer "F.Cu") (net "+3V3"))
@@
 (segment (start 90.950000 93.492711) (end 91.350000 92.800000) (width 0.1778) (layer "F.Cu") (net "SCL"))
 (segment (start 91.350000 92.800000) (end 93.100000 92.736800) (width 0.1778) (layer "F.Cu") (net "SCL"))
-(via (at 87.900000 93.600000) (size 0.604) (drill 0.35) (layers "F.Cu" "B.Cu") (net "GND"))
-(segment (start 87.900000 93.600000) (end 88.587306 93.492711) (width 0.3000) (layer "F.Cu") (net "GND"))
-(via (at 90.700000 91.650000) (size 0.604) (drill 0.35) (layers "F.Cu" "B.Cu") (net "GND"))
-(segment (start 90.700000 91.650000) (end 90.249806 92.330211) (width 0.3000) (layer "F.Cu") (net "GND"))
+(via (at 87.900000 93.800000) (size 0.604) (drill 0.35) (layers "F.Cu" "B.Cu") (net "GND"))
+(segment (start 87.900000 93.800000) (end 88.587306 93.492711) (width 0.3000) (layer "F.Cu") (net "GND"))
 (segment (start 90.249806 92.330211) (end 89.749806 92.330211) (width 0.3000) (layer "F.Cu") (net "GND"))
 (segment (start 89.749806 92.330211) (end 89.249806 92.330211) (width 0.3000) (layer "F.Cu") (net "GND"))
@@
 (segment (start 92.850000 94.000000) (end 92.850000 93.350000) (width 0.2500) (layer "F.Cu") (net "+3V3"))
 (segment (start 92.004083 94.507669) (end 91.450000 94.200000) (width 0.2500) (layer "F.Cu") (net "+3V3"))
-(segment (start 91.450000 94.200000) (end 90.412306 93.992711) (width 0.2500) (layer "F.Cu") (net "+3V3"))
+(segment (start 91.450000 94.200000) (end 90.700000 94.200000) (width 0.2500) (layer "F.Cu") (net "+3V3"))
 (segment (start 89.249806 94.655211) (end 89.249806 94.250000) (width 0.1778) (layer "F.Cu") (net "/IMU_INT2"))
 (segment (start 89.249806 94.250000) (end 89.619500 93.580900) (width 0.1778) (layer "F.Cu") (net "/IMU_INT2"))
@@
 (segment (start 93.100000 92.750000) (end 94.040000 92.310200) (width 0.1778) (layer "In2.Cu") (net "/IMU_INT2"))
 (via (at 89.619500 93.580900) (size 0.604) (drill 0.35) (layers "F.Cu" "B.Cu") (net "/IMU_INT2"))
-(via (at 87.850000 92.700000) (size 0.604) (drill 0.35) (layers "F.Cu" "B.Cu") (net "+3V3"))
-(segment (start 88.587306 92.992711) (end 87.850000 92.700000) (width 0.2500) (layer "F.Cu") (net "+3V3"))
-(via (at 88.150000 91.800000) (size 0.604) (drill 0.35) (layers "F.Cu" "B.Cu") (net "+3V3"))
-(segment (start 88.794835 91.491614) (end 88.150000 91.800000) (width 0.1778) (layer "F.Cu") (net "+3V3"))
+(via (at 87.950000 92.550000) (size 0.604) (drill 0.35) (layers "F.Cu" "B.Cu") (net "+3V3"))
+(segment (start 88.587306 92.992711) (end 87.950000 92.550000) (width 0.2500) (layer "F.Cu") (net "+3V3"))
+(via (at 88.794835 90.050000) (size 0.604) (drill 0.35) (layers "F.Cu" "B.Cu") (net "+3V3"))
+(segment (start 88.794835 91.491614) (end 88.794835 90.050000) (width 0.1778) (layer "F.Cu") (net "+3V3"))
 (segment (start 87.094469 95.226030) (end 88.000000 95.226030) (width 0.1778) (layer "F.Cu") (net "+3V3"))
 (segment (start 88.000000 95.226030) (end 88.749806 95.250000) (width 0.1778) (layer "F.Cu") (net "+3V3"))
-(segment (start 87.082668 93.109941) (end 87.850000 92.700000) (width 0.1778) (layer "F.Cu") (net "+3V3"))
-(segment (start 86.600000 93.109900) (end 87.082668 93.109941) (width 0.1778) (layer "F.Cu") (net "+3V3"))
+(segment (start 87.082668 92.609941) (end 87.950000 92.550000) (width 0.1778) (layer "F.Cu") (net "+3V3"))
+(segment (start 86.600000 93.109900) (end 87.082668 92.609941) (width 0.1778) (layer "F.Cu") (net "+3V3"))
 (segment (start 88.393800 90.500000) (end 88.794835 91.491614) (width 0.1778) (layer "F.Cu") (net "+3V3"))
-(segment (start 87.850000 92.700000) (end 88.200000 92.900000) (width 0.4000) (layer "In2.Cu") (net "+3V3"))
-(segment (start 88.150000 91.800000) (end 88.200000 92.900000) (width 0.4000) (layer "In2.Cu") (net "+3V3"))
+(segment (start 87.950000 92.550000) (end 88.200000 92.900000) (width 0.4000) (layer "In2.Cu") (net "+3V3"))
+(segment (start 88.794835 90.050000) (end 88.794835 92.000000) (width 0.4000) (layer "In2.Cu") (net "+3V3"))
 (segment (start 88.200000 92.900000) (end 88.600000 93.200000) (width 0.4000) (layer "In2.Cu") (net "+3V3"))
 (segment (start 88.600000 93.200000) (end 88.700000 94.300000) (width 0.4000) (layer "In2.Cu") (net "+3V3"))
@@
 (segment (start 92.400000 94.200000) (end 92.800000 93.600000) (width 0.4000) (layer "In2.Cu") (net "+3V3"))
 (segment (start 92.800000 93.600000) (end 92.850000 93.350000) (width 0.4000) (layer "In2.Cu") (net "+3V3"))
+(via (at 87.094469 93.550000) (size 0.604) (drill 0.35) (layers "F.Cu" "B.Cu") (net "SCL"))
+(via (at 91.020000 93.492711) (size 0.604) (drill 0.35) (layers "F.Cu" "B.Cu") (net "SCL"))
+(via (at 87.000000 90.050000) (size 0.604) (drill 0.35) (layers "F.Cu" "B.Cu") (net "SDA"))
+(via (at 90.700000 91.650000) (size 0.604) (drill 0.35) (layers "F.Cu" "B.Cu") (net "SDA"))
+(via (at 87.970000 91.720000) (size 0.604) (drill 0.35) (layers "F.Cu" "B.Cu") (net "INT"))
+(via (at 91.800000 92.140000) (size 0.604) (drill 0.35) (layers "F.Cu" "B.Cu") (net "INT"))
+(segment (start 89.749806 92.330211) (end 89.810835 91.491614) (width 0.3000) (layer "F.Cu") (net "GND"))
+(segment (start 88.794835 92.000000) (end 88.200000 92.900000) (width 0.4000) (layer "In2.Cu") (net "+3V3"))
+(segment (start 90.700000 94.200000) (end 90.412306 93.992711) (width 0.2500) (layer "F.Cu") (net "+3V3"))
+(segment (start 87.094469 94.210030) (end 87.094469 93.550000) (width 0.1778) (layer "F.Cu") (net "SCL"))
+(segment (start 87.082668 91.593941) (end 87.000000 90.050000) (width 0.1778) (layer "F.Cu") (net "SDA"))
+(segment (start 90.412306 92.992711) (end 90.700000 92.992711) (width 0.1778) (layer "F.Cu") (net "SDA"))
+(segment (start 90.700000 92.992711) (end 90.700000 91.650000) (width 0.1778) (layer "F.Cu") (net "SDA"))
+(segment (start 88.749806 92.330211) (end 88.300000 92.030000) (width 0.1778) (layer "F.Cu") (net "INT"))
+(segment (start 88.300000 92.030000) (end 87.970000 91.720000) (width 0.1778) (layer "F.Cu") (net "INT"))
+(segment (start 87.094469 93.550000) (end 87.100000 93.170000) (width 0.1778) (layer "B.Cu") (net "SCL"))
+(segment (start 87.100000 93.170000) (end 88.700000 93.170000) (width 0.1778) (layer "B.Cu") (net "SCL"))
+(segment (start 88.700000 93.170000) (end 89.000000 92.950000) (width 0.1778) (layer "B.Cu") (net "SCL"))
+(segment (start 89.000000 92.950000) (end 90.400000 92.950000) (width 0.1778) (layer "B.Cu") (net "SCL"))
+(segment (start 90.400000 92.950000) (end 91.020000 93.492711) (width 0.1778) (layer "B.Cu") (net "SCL"))
+(segment (start 87.000000 90.050000) (end 87.000000 89.570000) (width 0.1778) (layer "In2.Cu") (net "SDA"))
+(segment (start 87.000000 89.570000) (end 88.400000 89.570000) (width 0.1778) (layer "In2.Cu") (net "SDA"))
+(segment (start 88.400000 89.570000) (end 88.550000 89.420000) (width 0.1778) (layer "In2.Cu") (net "SDA"))
+(segment (start 88.550000 89.420000) (end 89.500000 89.420000) (width 0.1778) (layer "In2.Cu") (net "SDA"))
+(segment (start 89.500000 89.420000) (end 89.500000 91.650000) (width 0.1778) (layer "In2.Cu") (net "SDA"))
+(segment (start 89.500000 91.650000) (end 90.700000 91.650000) (width 0.1778) (layer "In2.Cu") (net "SDA"))
+(segment (start 90.700000 91.650000) (end 93.100000 91.377100) (width 0.1778) (layer "B.Cu") (net "SDA"))
+(segment (start 87.970000 91.720000) (end 89.000000 92.100000) (width 0.1778) (layer "B.Cu") (net "INT"))
+(segment (start 89.000000 92.100000) (end 90.000000 92.500000) (width 0.1778) (layer "B.Cu") (net "INT"))
+(segment (start 90.000000 92.500000) (end 91.000000 92.500000) (width 0.1778) (layer "B.Cu") (net "INT"))
+(segment (start 91.000000 92.500000) (end 91.800000 92.140000) (width 0.1778) (layer "B.Cu") (net "INT"))
+(segment (start 91.800000 92.140000) (end 92.000000 91.400000) (width 0.1778) (layer "F.Cu") (net "INT"))
+(segment (start 92.000000 91.400000) (end 93.100000 91.400000) (width 0.1778) (layer "F.Cu") (net "INT"))
 )
